File: Controller/kicad/level.kicad_sch (KiCad schematic)
At the start: 38 parts, among them Q1 2N7002, Q10 MMBT5551L, Q11 2N7002, Q12 2N7002, Q2 2N7002, Q3 AO3401A, Q4 MMBT5551L, Q5 2N7002, Q6 2N7002, Q7 AO3401A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

Commit message: Tweaked board to allow for JLCPCB standard assembly.  Needed fiducials and 5mm rail clearance top and bottom.  Also fixed silkscreen mistake
Parts:
- Q1, Q10, Q11, Q12, Q2, Q3, Q4, Q5, Q6, Q7, Q8, Q9: JLCPCB_CORRECTION (none) -> 0; 0; 180
Changed lines of the file:
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@@
+      (effects (font (size 1.27 1.27)) hide)
+    )
+    (property "JLCPCB_CORRECTION" "0; 0; 180" (id 5) (at 54.61 120.65 0)
       (effects (font (size 1.27 1.27)) hide)
     )
@@
       (effects (font (size 1.27 1.27)) hide)
     )
+    (property "JLCPCB_CORRECTION" "0; 0; 180" (id 5) (at 242.57 87.63 0)
+      (effects (font (size 1.27 1.27)) hide)
+    )
     (pin "1")
     (pin "2")
@@
       (effects (font (size 1.27 1.27)) hide)
     )
+    (property "JLCPCB_CORRECTION" "0; 0; 180" (id 5) (at 54.61 92.71 0)
+      (effects (font (size 1.27 1.27)) hide)
+    )
     (pin "1")
     (pin "2")
@@
     )
     (property "LCSC" "C2145" (id 4) (at 234.95 49.53 0)
+      (effects (font (size 1.27 1.27)) hide)
+    )
+    (property "JLCPCB_CORRECTION" "0; 0; 180" (id 5) (at 234.95 49.53 0)
       (effects (font (size 1.27 1.27)) hide)
     )
@@
       (effects (font (size 1.27 1.27)) hide)
     )
+    (property "JLCPCB_CORRECTION" "0; 0; 180" (id 5) (at 130.81 92.71 0)
+      (effects (font (size 1.27 1.27)) hide)
+    )
     (pin "1")
     (pin "2")
@@
     )
     (property "LCSC" "C15127" (id 4) (at 242.57 36.83 0)
+      (effects (font (size 1.27 1.27)) hide)
+    )
+    (property "JLCPCB_CORRECTION" "0; 0; 180" (id 5) (at 242.57 36.83 0)
       (effects (font (size 1.27 1.27)) hide)
     )
@@
       (effects (font (size 1.27 1.27)) hide)
     )
+    (property "JLCPCB_CORRECTION" "0; 0; 180" (id 5) (at 55.88 35.56 0)
+      (effects (font (size 1.27 1.27)) hide)
+    )
     (pin "1")
     (pin "2")
@@
       (effects (font (size 1.27 1.27)) hide)
     )
+    (property "JLCPCB_CORRECTION" "0; 0; 180" (id 5) (at 130.81 35.56 0)
+      (effects (font (size 1.27 1.27)) hide)
+    )
     (pin "1")
     (pin "2")
@@
       (effects (font (size 1.27 1.27)) hide)
     )
+    (property "JLCPCB_CORRECTION" "0; 0; 180" (id 5) (at 130.81 63.5 0)
+      (effects (font (size 1.27 1.27)) hide)
+    )
     (pin "1")
     (pin "2")
@@
       (effects (font (size 1.27 1.27)) hide)
     )
+    (property "JLCPCB_CORRECTION" "0; 0; 180" (id 5) (at 55.88 63.5 0)
+      (effects (font (size 1.27 1.27)) hide)
+    )
     (pin "1")
     (pin "2")
@@
     )
     (property "LCSC" "C2145" (id 4) (at 234.95 100.33 0)
+      (effects (font (size 1.27 1.27)) hide)
+    )
+    (property "JLCPCB_CORRECTION" "0; 0; 180" (id 5) (at 234.95 100.33 0)
       (effects (font (size 1.27 1.27)) hide)
     )
@@
       (effects (font (size 1.27 1.27)) hide)
     )
+    (property "JLCPCB_CORRECTION" "0; 0; 180" (id 5) (at 130.81 120.65 0)
+      (effects (font (size 1.27 1.27)) hide)
+    )

Commit message: Updated schematics based on issues and improvements from the prototype board
Parts:
- added R? (x2): 10k, Resistor_SMD:R_0603_1608Metric, symbol Device:R
Connections:
- net +3V3: now also R?.2, R?.2; no longer SW3.2, SW4.2
- new net: R?.1, SW4.2
- new net: R?.1, SW3.2
Changed lines of the file:
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@@
     (pin "2")
   )
-  (symbol (lib_id "power:+3V3") (at 220.98 35.56 0) (unit 1)
-    (in_bom yes) (on_board yes) (fields_autoplaced)
-    (property "Reference" "#PWR058" (id 0) (at 220.98 39.37 0)
-      (effects (font (size 1.27 1.27)) hide)
-    )
-    (property "Value" "+3V3" (id 1) (at 220.98 30.48 0))
-    (property "Footprint" "" (id 2) (at 220.98 35.56 0)
-      (effects (font (size 1.27 1.27)) hide)
-    )
-    (property "Datasheet" "" (id 3) (at 220.98 35.56 0)
+  (symbol (lib_id "power:+3V3") (at 220.98 27.94 0) (unit 1)
+    (in_bom yes) (on_board yes) (fields_autoplaced)
+    (property "Reference" "#PWR058" (id 0) (at 220.98 31.75 0)
+      (effects (font (size 1.27 1.27)) hide)
+    )
+    (property "Value" "+3V3" (id 1) (at 220.98 22.86 0))
+    (property "Footprint" "" (id 2) (at 220.98 27.94 0)
+      (effects (font (size 1.27 1.27)) hide)
+    )
+    (property "Datasheet" "" (id 3) (at 220.98 27.94 0)
       (effects (font (size 1.27 1.27)) hide)
     )
@@
     (pin "1")
   )
-  (symbol (lib_id "power:+3V3") (at 220.98 86.36 0) (unit 1)
-    (in_bom yes) (on_board yes) (fields_autoplaced)
-    (property "Reference" "#PWR065" (id 0) (at 220.98 90.17 0)
-      (effects (font (size 1.27 1.27)) hide)
-    )
-    (property "Value" "+3V3" (id 1) (at 220.98 81.28 0))
-    (property "Footprint" "" (id 2) (at 220.98 86.36 0)
-      (effects (font (size 1.27 1.27)) hide)
-    )
-    (property "Datasheet" "" (id 3) (at 220.98 86.36 0)
+  (symbol (lib_id "power:+3V3") (at 220.98 78.74 0) (unit 1)
+    (in_bom yes) (on_board yes) (fields_autoplaced)
+    (property "Reference" "#PWR065" (id 0) (at 220.98 82.55 0)
+      (effects (font (size 1.27 1.27)) hide)
+    )
+    (property "Value" "+3V3" (id 1) (at 220.98 73.66 0))
+    (property "Footprint" "" (id 2) (at 220.98 78.74 0)
+      (effects (font (size 1.27 1.27)) hide)
+    )
+    (property "Datasheet" "" (id 3) (at 220.98 78.74 0)
       (effects (font (size 1.27 1.27)) hide)
     )
@@
     (pin "1")
   )
+  (symbol (lib_id "Device:R") (at 220.98 31.75 180) (unit 1)
+    (in_bom yes) (on_board yes) (fields_autoplaced)
+    (property "Reference" "R?" (id 0) (at 223.52 30.4799 0)
+      (effects (font (size 1.27 1.27)) (justify right))
+    )
+    (property "Value" "10k" (id 1) (at 223.52 33.0199 0)
+      (effects (font (size 1.27 1.27)) (justify right))
+    )
+    (property "Footprint" "Resistor_SMD:R_0603_1608Metric" (id 2) (at 222.758 31.75 90)
+      (effects (font (size 1.27 1.27)) hide)
+    )
+    (property "Datasheet" "~" (id 3) (at 220.98 31.75 0)
+      (effects (font (size 1.27 1.27)) hide)
+    )
+    (property "LCSC" "C25804" (id 4) (at 220.98 31.75 0)
+      (effects (font (size 1.27 1.27)) hide)
+    )
+    (pin "1")
+    (pin "2")
+  )
   (symbol (lib_id "power:+3V3") (at 46.99 30.48 0) (unit 1)
     (in_bom yes) (on_board yes) (fields_autoplaced)
@@
     (pin "1")
   )
+  (symbol (lib_id "Device:R") (at 220.98 82.55 180) (unit 1)
+    (in_bom yes) (on_board yes) (fields_autoplaced)
+    (property "Reference" "R?" (id 0) (at 223.52 81.2799 0)
+      (effects (font (size 1.27 1.27)) (justify right))
+    )
+    (property "Value" "10k" (id 1) (at 223.52 83.8199 0)
+      (effects (font (size 1.27 1.27)) (justify right))
+    )
+    (property "Footprint" "Resistor_SMD:R_0603_1608Metric" (id 2) (at 222.758 82.55 90)
+      (effects (font (size 1.27 1.27)) hide)
+    )
+    (property "Datasheet" "~" (id 3) (at 220.98 82.55 0)
+      (effects (font (size 1.27 1.27)) hide)
+    )
+    (property "LCSC" "C25804" (id 4) (at 220.98 82.55 0)
+      (effects (font (size 1.27 1.27)) hide)
+    )
+    (pin "1")
+    (pin "2")
+  )
 )

Commit message: Pre-production check-in
Parts:
- gave numbers to parts that had none: 2
Connections:
- net +BATT renamed +12V
Changed lines of the file:
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@@
   (junction (at 45.72 123.19) (diameter 0) (color 0 0 0 0)
   )
+  (junction (at 237.49 80.01) (diameter 0) (color 0 0 0 0)
+  )
   (junction (at 121.92 58.42) (diameter 0) (color 0 0 0 0)
   )
@@
   (junction (at 63.5 123.19) (diameter 0) (color 0 0 0 0)
   )
+  (junction (at 139.7 123.19) (diameter 0) (color 0 0 0 0)
+  )
+  (junction (at 220.98 49.53) (diameter 0) (color 0 0 0 0)
+  )
+  (junction (at 220.98 100.33) (diameter 0) (color 0 0 0 0)
+  )
+  (junction (at 63.5 95.25) (diameter 0) (color 0 0 0 0)
+  )
+  (junction (at 45.72 95.25) (diameter 0) (color 0 0 0 0)
+  )
+  (junction (at 121.92 30.48) (diameter 0) (color 0 0 0 0)
+  )
+  (junction (at 139.7 38.1) (diameter 0) (color 0 0 0 0)
+  )
+  (junction (at 45.72 87.63) (diameter 0) (color 0 0 0 0)
+  )
+  (junction (at 237.49 36.83) (diameter 0) (color 0 0 0 0)
+  )
+  (junction (at 121.92 95.25) (diameter 0) (color 0 0 0 0)
+  )
+  (junction (at 139.7 95.25) (diameter 0) (color 0 0 0 0)
+  )
+  (junction (at 64.77 66.04) (diameter 0) (color 0 0 0 0)
+  )
+  (junction (at 46.99 30.48) (diameter 0) (color 0 0 0 0)
+  )
+  (junction (at 121.92 66.04) (diameter 0) (color 0 0 0 0)
+  )
+  (junction (at 121.92 123.19) (diameter 0) (color 0 0 0 0)
+  )
+  (junction (at 139.7 66.04) (diameter 0) (color 0 0 0 0)
+  )
+  (junction (at 237.49 87.63) (diameter 0) (color 0 0 0 0)
+  )
+  (junction (at 46.99 58.42) (diameter 0) (color 0 0 0 0)
+  )
   (junction (at 237.49 29.21) (diameter 0) (color 0 0 0 0)
-  )
-  (junction (at 139.7 123.19) (diameter 0) (color 0 0 0 0)
-  )
-  (junction (at 220.98 49.53) (diameter 0) (color 0 0 0 0)
-  )
-  (junction (at 220.98 100.33) (diameter 0) (color 0 0 0 0)
-  )
-  (junction (at 63.5 95.25) (diameter 0) (color 0 0 0 0)
-  )
-  (junction (at 45.72 95.25) (diameter 0) (color 0 0 0 0)
-  )
-  (junction (at 121.92 30.48) (diameter 0) (color 0 0 0 0)
-  )
-  (junction (at 139.7 38.1) (diameter 0) (color 0 0 0 0)
-  )
-  (junction (at 45.72 87.63) (diameter 0) (color 0 0 0 0)
-  )
-  (junction (at 237.49 36.83) (diameter 0) (color 0 0 0 0)
-  )
-  (junction (at 121.92 95.25) (diameter 0) (color 0 0 0 0)
-  )
-  (junction (at 139.7 95.25) (diameter 0) (color 0 0 0 0)
-  )
-  (junction (at 64.77 66.04) (diameter 0) (color 0 0 0 0)
-  )
-  (junction (at 46.99 30.48) (diameter 0) (color 0 0 0 0)
-  )
-  (junction (at 237.49 80.01) (diameter 0) (color 0 0 0 0)
-  )
-  (junction (at 121.92 66.04) (diameter 0) (color 0 0 0 0)
-  )
-  (junction (at 121.92 123.19) (diameter 0) (color 0 0 0 0)
-  )
-  (junction (at 139.7 66.04) (diameter 0) (color 0 0 0 0)
-  )
-  (junction (at 237.49 87.63) (diameter 0) (color 0 0 0 0)
-  )
-  (junction (at 46.99 58.42) (diameter 0) (color 0 0 0 0)
   )
   (junction (at 45.72 115.57) (diameter 0) (color 0 0 0 0)
@@
     (pin "3")
   )
+  (symbol (lib_id "power:+12V") (at 237.49 29.21 0) (unit 1)
+    (in_bom yes) (on_board yes) (fields_autoplaced)
+    (property "Reference" "#PWR0106" (id 0) (at 237.49 33.02 0)
+      (effects (font (size 1.27 1.27)) hide)
+    )
+    (property "Value" "+12V" (id 1) (at 237.49 24.13 0))
+    (property "Footprint" "" (id 2) (at 237.49 29.21 0)
+      (effects (font (size 1.27 1.27)) hide)
+    )
+    (property "Datasheet" "" (id 3) (at 237.49 29.21 0)
+      (effects (font (size 1.27 1.27)) hide)
+    )
+    (pin "1")
+  )
   (symbol (lib_id "Device:Fuse") (at 251.46 92.71 270) (unit 1)
     (in_bom yes) (on_board yes)
@@
       (effects (font (size 1.27 1.27)) hide)
     )
-    (property "Datasheet" "https://datasheet.lcsc.com/lcsc/2002271431_XKB-Connectivity-TS-1187A-B-A-B_C318884.pdf" (id 3) (at 215.9 91.44 0)
+    (property "Datasheet" "~" (id 3) (at 215.9 91.44 0)
       (effects (font (size 1.27 1.27)) hide)
     )
@@
     )
     (property "Datasheet" "" (id 3) (at 64.77 30.48 0)
-      (effects (font (size 1.27 1.27)) hide)
-    )
-    (pin "1")
-  )
-  (symbol (lib_id "Power:V_BATT") (at 237.49 29.21 0) (unit 1)
-    (in_bom yes) (on_board yes) (fields_autoplaced)
-    (property "Reference" "#PWR053" (id 0) (at 237.49 33.02 0)
-      (effects (font (size 1.27 1.27)) hide)
-    )
-    (property "Value" "V_BATT" (id 1) (at 237.49 24.13 0))
-    (property "Footprint" "" (id 2) (at 237.49 29.21 0)
-      (effects (font (size 1.27 1.27)) hide)
-    )
-    (property "Datasheet" "" (id 3) (at 237.49 29.21 0)
       (effects (font (size 1.27 1.27)) hide)
     )
@@
       (effects (font (size 1.27 1.27) italic) (justify left) hide)
     )
-    (property "Datasheet" "https://datasheet.lcsc.com/lcsc/1810171817_Alpha---Omega-Semicon-AO3401A_C15127.pdf" (id 3) (at 242.57 87.63 0)
+    (property "Datasheet" "http://www.aosmd.com/pdfs/datasheet/AO3401A.pdf" (id 3) (at 242.57 87.63 0)
       (effects (font (size 1.27 1.27)) (justify left) hide)
     )
@@
     (pin "2")
   )
+  (symbol (lib_id "power:+12V") (at 237.49 80.01 0) (unit 1)
+    (in_bom yes) (on_board yes) (fields_autoplaced)
+    (property "Reference" "#PWR0105" (id 0) (at 237.49 83.82 0)
+      (effects (font (size 1.27 1.27)) hide)
+    )
+    (property "Value" "+12V" (id 1) (at 237.49 74.93 0))
+    (property "Footprint" "" (id 2) (at 237.49 80.01 0)
+      (effects (font (size 1.27 1.27)) hide)
+    )
+    (property "Datasheet" "" (id 3) (at 237.49 80.01 0)
+      (effects (font (size 1.27 1.27)) hide)
+    )
+    (pin "1")
+  )
   (symbol (lib_id "Device:R") (at 63.5 119.38 0) (unit 1)
     (in_bom yes) (on_board yes)
@@
       (effects (font (size 1.27 1.27) italic) (justify left) hide)
     )
-    (property "Datasheet" "https://datasheet.lcsc.com/lcsc/1810190020_Jiangsu-Changjing-Electronics-Technology-Co---Ltd--MMBT5551_C2145.pdf" (id 3) (at 234.95 49.53 0)
+    (property "Datasheet" "www.onsemi.com/pub/Collateral/MMBT5550LT1-D.PDF" (id 3) (at 234.95 49.53 0)
       (effects (font (size 1.27 1.27)) (justify left) hide)
     )
@@
       (effects (font (size 1.27 1.27) italic) (justify left) hide)
     )
-    (property "Datasheet" "https://datasheet.lcsc.com/lcsc/1810171817_Alpha---Omega-Semicon-AO3401A_C15127.pdf" (id 3) (at 242.57 36.83 0)
+    (property "Datasheet" "http://www.aosmd.com/pdfs/datasheet/AO3401A.pdf" (id 3) (at 242.57 36.83 0)
       (effects (font (size 1.27 1.27)) (justify left) hide)
     )
@@
     (pin "2")
     (pin "3")
-  )
-  (symbol (lib_id "Power:V_BATT") (at 237.49 80.01 0) (unit 1)
-    (in_bom yes) (on_board yes) (fields_autoplaced)
-    (property "Reference" "#PWR064" (id 0) (at 237.49 83.82 0)
-      (effects (font (size 1.27 1.27)) hide)
-    )
-    (property "Value" "V_BATT" (id 1) (at 237.49 74.93 0))
-    (property "Footprint" "" (id 2) (at 237.49 80.01 0)
-      (effects (font (size 1.27 1.27)) hide)
-    )
-    (property "Datasheet" "" (id 3) (at 237.49 80.01 0)
-      (effects (font (size 1.27 1.27)) hide)
-    )
-    (pin "1")
   )
   (symbol (lib_id "Transistor_FET:2N7002") (at 55.88 35.56 270) (unit 1)
@@
       (effects (font (size 1.27 1.27) italic) (justify left) hide)
     )
-    (property "Datasheet" "https://datasheet.lcsc.com/lcsc/1810151612_Jiangsu-Changjing-Electronics-Technology-Co---Ltd--2N7002_C8545.pdf" (id 3) (at 55.88 35.56 0)
+    (property "Datasheet" "https://www.onsemi.com/pub/Collateral/NDS7002A-D.PDF" (id 3) (at 55.88 35.56 0)
       (effects (font (size 1.27 1.27)) (justify left) hide)
     )
@@
       (effects (font (size 1.27 1.27)) hide)
     )
-    (property "Datasheet" "https://datasheet.lcsc.com/lcsc/2002271431_XKB-Connectivity-TS-1187A-B-A-B_C318884.pdf" (id 3) (at 215.9 40.64 0)
+    (property "Datasheet" "~" (id 3) (at 215.9 40.64 0)
       (effects (font (size 1.27 1.27)) hide)
     )
@@
       (effects (font (size 1.27 1.27) italic) (justify left) hide)
     )
-    (property "Datasheet" "https://datasheet.lcsc.com/lcsc/1810190020_Jiangsu-Changjing-Electronics-Technology-Co---Ltd--MMBT5551_C2145.pdf" (id 3) (at 234.95 100.33 0)
+    (property "Datasheet" "www.onsemi.com/pub/Collateral/MMBT5550LT1-D.PDF" (id 3) (at 234.95 100.33 0)
       (effects (font (size 1.27 1.27)) (justify left) hide)
     )
@@
   (symbol (lib_id "Device:R") (at 220.98 31.75 180) (unit 1)
     (in_bom yes) (on_board yes) (fields_autoplaced)
-    (property "Reference" "R?" (id 0) (at 223.52 30.4799 0)
+    (property "Reference" "R41" (id 0) (at 223.52 30.4799 0)
       (effects (font (size 1.27 1.27)) (justify right))
     )
@@
   (symbol (lib_id "Device:R") (at 220.98 82.55 180) (unit 1)
     (in_bom yes) (on_board yes) (fields_autoplaced)
-    (property "Reference" "R?" (id 0) (at 223.52 81.2799 0)
+    (property "Reference" "R42" (id 0) (at 223.52 81.2799 0)
       (effects (font (size 1.27 1.27)) (justify right))
     )
