File: Controller/kicad/power.kicad_sch (KiCad schematic)
At the start: 15 parts, among them J10 BATTERY, J9 V_IN, U1 MP1584, U2 LM317_TO-252, U3 AMS1117-3.3

Commit message: Tweaked board to allow for JLCPCB standard assembly.  Needed fiducials and 5mm rail clearance top and bottom.  Also fixed silkscreen mistake
Parts:
- C1, C2, U3: JLCPCB_CORRECTION (none) -> 0; 0; 180
Changed lines of the file:
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@@
+      (effects (font (size 1.27 1.27)) hide)
+    )
+    (property "JLCPCB_CORRECTION" "0; 0; 180" (id 5) (at 213.36 90.17 0)
       (effects (font (size 1.27 1.27)) hide)
     )
@@
     )
     (property "LCSC" "C6186" (id 4) (at 223.52 86.36 0)
+      (effects (font (size 1.27 1.27)) hide)
+    )
+    (property "JLCPCB_CORRECTION" "0; 0; 180" (id 5) (at 223.52 86.36 0)
       (effects (font (size 1.27 1.27)) hide)
     )
@@
       (effects (font (size 1.27 1.27)) hide)
     )
+    (property "JLCPCB_CORRECTION" "0; 0; 180" (id 5) (at 233.68 90.17 0)
+      (effects (font (size 1.27 1.27)) hide)
+    )

Commit message: Updated schematics based on issues and improvements from the prototype board
Parts:
- added J?: Jack-DC, symbol Connector:Jack-DC
Connections:
- net GND: now also J?.2
- net at F1.2, J9.1 (Pin_1): now also J?.1
Other:
- moved on the sheet: D1, F1
Changed lines of the file:
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@@
   (junction (at 83.82 163.83) (diameter 0) (color 0 0 0 0)
   )
+  (junction (at 142.24 86.36) (diameter 0) (color 0 0 0 0)
+  )
+  (junction (at 124.46 86.36) (diameter 0) (color 0 0 0 0)
+  )
+  (junction (at 163.83 86.36) (diameter 0) (color 0 0 0 0)
+  )
+  (junction (at 113.03 93.98) (diameter 0) (color 0 0 0 0)
+  )
+  (junction (at 62.23 163.83) (diameter 0) (color 0 0 0 0)
+  )
+  (junction (at 179.07 96.52) (diameter 0) (color 0 0 0 0)
+  )
+  (junction (at 201.93 86.36) (diameter 0) (color 0 0 0 0)
+  )
+  (junction (at 213.36 86.36) (diameter 0) (color 0 0 0 0)
+  )
+  (junction (at 116.84 93.98) (diameter 0) (color 0 0 0 0)
+  )
+  (junction (at 116.84 86.36) (diameter 0) (color 0 0 0 0)
+  )
+  (junction (at 91.44 86.36) (diameter 0) (color 0 0 0 0)
+  )
+  (junction (at 62.23 171.45) (diameter 0) (color 0 0 0 0)
+  )
+  (junction (at 55.88 86.36) (diameter 0) (color 0 0 0 0)
+  )
+  (junction (at 233.68 86.36) (diameter 0) (color 0 0 0 0)
+  )
+  (junction (at 223.52 93.98) (diameter 0) (color 0 0 0 0)
+  )
   (junction (at 82.55 86.36) (diameter 0) (color 0 0 0 0)
   )
-  (junction (at 142.24 86.36) (diameter 0) (color 0 0 0 0)
-  )
-  (junction (at 124.46 86.36) (diameter 0) (color 0 0 0 0)
-  )
-  (junction (at 163.83 86.36) (diameter 0) (color 0 0 0 0)
-  )
-  (junction (at 113.03 93.98) (diameter 0) (color 0 0 0 0)
-  )
-  (junction (at 62.23 163.83) (diameter 0) (color 0 0 0 0)
-  )
-  (junction (at 179.07 96.52) (diameter 0) (color 0 0 0 0)
-  )
-  (junction (at 201.93 86.36) (diameter 0) (color 0 0 0 0)
-  )
-  (junction (at 213.36 86.36) (diameter 0) (color 0 0 0 0)
-  )
-  (junction (at 116.84 93.98) (diameter 0) (color 0 0 0 0)
-  )
-  (junction (at 116.84 86.36) (diameter 0) (color 0 0 0 0)
-  )
-  (junction (at 91.44 86.36) (diameter 0) (color 0 0 0 0)
-  )
-  (junction (at 62.23 171.45) (diameter 0) (color 0 0 0 0)
-  )
-  (junction (at 233.68 86.36) (diameter 0) (color 0 0 0 0)
-  )
-  (junction (at 223.52 93.98) (diameter 0) (color 0 0 0 0)
-  )
   (wire (pts (xy 201.93 60.96) (xy 201.93 86.36))
     (stroke (width 0) (type default) (color 0 0 0 0))
@@
     (stroke (width 0) (type default) (color 0 0 0 0))
   )
-  (wire (pts (xy 49.53 86.36) (xy 54.61 86.36))
+  (wire (pts (xy 49.53 86.36) (xy 55.88 86.36))
     (stroke (width 0) (type default) (color 0 0 0 0))
   )
@@
     (stroke (width 0) (type default) (color 0 0 0 0))
   )
+  (wire (pts (xy 74.93 86.36) (xy 82.55 86.36))
+    (stroke (width 0) (type default) (color 0 0 0 0))
+  )
   (wire (pts (xy 62.23 171.45) (xy 49.53 171.45))
     (stroke (width 0) (type default) (color 0 0 0 0))
@@
     (stroke (width 0) (type default) (color 0 0 0 0))
   )
+  (wire (pts (xy 55.88 86.36) (xy 59.69 86.36))
+    (stroke (width 0) (type default) (color 0 0 0 0))
+  )
   (wire (pts (xy 49.53 171.45) (xy 49.53 166.37))
     (stroke (width 0) (type default) (color 0 0 0 0))
@@
     (stroke (width 0) (type default) (color 0 0 0 0))
   )
-  (wire (pts (xy 69.85 86.36) (xy 82.55 86.36))
+  (wire (pts (xy 55.88 86.36) (xy 55.88 105.41))
     (stroke (width 0) (type default) (color 0 0 0 0))
   )
@@
     (effects (font (size 1.27 1.27)) (justify left bottom))
   )
-  (symbol (lib_id "Device:Fuse") (at 58.42 86.36 270) (unit 1)
+  (symbol (lib_id "Device:Fuse") (at 63.5 86.36 270) (unit 1)
     (in_bom yes) (on_board yes)
-    (property "Reference" "F1" (id 0) (at 53.34 88.9 90))
-    (property "Value" "2A" (id 1) (at 58.42 88.9 90))
-    (property "Footprint" "Fuse:Fuseholder_Cylinder-5x20mm_Schurter_0031_8201_Horizontal_Open" (id 2) (at 58.42 84.582 90)
-      (effects (font (size 1.27 1.27)) hide)
-    )
-    (property "Datasheet" "~" (id 3) (at 58.42 86.36 0)
-      (effects (font (size 1.27 1.27)) hide)
-    )
-    (property "BUY" "C3130" (id 4) (at 58.42 86.36 0)
+    (property "Reference" "F1" (id 0) (at 58.42 88.9 90))
+    (property "Value" "2A" (id 1) (at 63.5 88.9 90))
+    (property "Footprint" "Fuse:Fuseholder_Cylinder-5x20mm_Schurter_0031_8201_Horizontal_Open" (id 2) (at 63.5 84.582 90)
+      (effects (font (size 1.27 1.27)) hide)
+    )
+    (property "Datasheet" "~" (id 3) (at 63.5 86.36 0)
+      (effects (font (size 1.27 1.27)) hide)
+    )
+    (property "BUY" "C3130" (id 4) (at 63.5 86.36 0)
       (effects (font (size 1.27 1.27)) hide)
     )
@@
     (pin "1")
   )
-  (symbol (lib_id "Device:D_Schottky") (at 66.04 86.36 0) (mirror y) (unit 1)
-    (in_bom yes) (on_board yes) (fields_autoplaced)
-    (property "Reference" "D1" (id 0) (at 66.3575 80.01 0))
-    (property "Value" "SS210" (id 1) (at 66.3575 82.55 0))
-    (property "Footprint" "Diode_SMD:D_SMA" (id 2) (at 66.04 86.36 0)
-      (effects (font (size 1.27 1.27)) hide)
-    )
-    (property "Datasheet" "https://datasheet.lcsc.com/lcsc/1811071613_MDD-Microdiode-Electronics--SS210_C14996.pdf" (id 3) (at 66.04 86.36 0)
-      (effects (font (size 1.27 1.27)) hide)
-    )
-    (property "LCSC" "C14996" (id 4) (at 66.04 86.36 0)
+  (symbol (lib_id "Device:D_Schottky") (at 71.12 86.36 0) (mirror y) (unit 1)
+    (in_bom yes) (on_board yes) (fields_autoplaced)
+    (property "Reference" "D1" (id 0) (at 71.4375 80.01 0))
+    (property "Value" "SS210" (id 1) (at 71.4375 82.55 0))
+    (property "Footprint" "Diode_SMD:D_SMA" (id 2) (at 71.12 86.36 0)
+      (effects (font (size 1.27 1.27)) hide)
+    )
+    (property "Datasheet" "https://datasheet.lcsc.com/lcsc/1811071613_MDD-Microdiode-Electronics--SS210_C14996.pdf" (id 3) (at 71.12 86.36 0)
+      (effects (font (size 1.27 1.27)) hide)
+    )
+    (property "LCSC" "C14996" (id 4) (at 71.12 86.36 0)
       (effects (font (size 1.27 1.27)) hide)
     )
@@
     (pin "4")
   )
+  (symbol (lib_id "Connector:Jack-DC") (at 48.26 107.95 0) (unit 1)
+    (in_bom yes) (on_board yes) (fields_autoplaced)
+    (property "Reference" "J?" (id 0) (at 48.26 99.06 0))
+    (property "Value" "Jack-DC" (id 1) (at 48.26 101.6 0))
+    (property "Footprint" "" (id 2) (at 49.53 108.966 0)
+      (effects (font (size 1.27 1.27)) hide)
+    )
+    (property "Datasheet" "~" (id 3) (at 49.53 108.966 0)
+      (effects (font (size 1.27 1.27)) hide)
+    )
+    (pin "1")
+    (pin "2")
+  )
   (symbol (lib_id "Connector:Screw_Terminal_01x02") (at 44.45 163.83 0) (mirror y) (unit 1)
     (in_bom yes) (on_board yes) (fields_autoplaced)
@@
       (effects (font (size 1.27 1.27)) hide)
     )
+    (pin "1")
+  )
+  (symbol (lib_id "power:GND") (at 55.88 110.49 0) (unit 1)
+    (in_bom yes) (on_board yes) (fields_autoplaced)
+    (property "Reference" "#PWR?" (id 0) (at 55.88 116.84 0)
+      (effects (font (size 1.27 1.27)) hide)
+    )
+    (property "Value" "GND" (id 1) (at 55.88 115.57 0))
+    (property "Footprint" "" (id 2) (at 55.88 110.49 0)
+      (effects (font (size 1.27 1.27)) hide)
+    )
+    (property "Datasheet" "" (id 3) (at 55.88 110.49 0)
+      (effects (font (size 1.27 1.27)) hide)
+    )

Commit message: Pre-production check-in
Parts:
- J10, J9: footprint TerminalBlock_Phoenix:TerminalBlock_Phoenix_MPT-0,5-2-2.54_1x02_P2.54mm_Horizontal -> Connector_PinHeader_2.54mm:PinHeader_1x02_P2.54mm_Horizontal
- J14: renamed from J?; footprint (none) -> Connector_BarrelJack:BarrelJack_Horizontal
- R2: BUY C841782 -> (none); LCSC (none) -> C841782
Connections:
- net V_BATT: now reaches D2.2 (A), D3.1 (K), F2.1, R2.2, R3.1
- net +BATT renamed +12V
