File: Controller/kicad/rLab_Door.kicad_sch (KiCad schematic)
At the start: 9 parts, among them J1 ACT_1, J2 ACT_2, J3 NPX_1, J4 NPX_2, J5 WIEGAND KEYPAD, J6 NFC SERIAL, J7 I2C DISPLAY, J8 TAMPER

Commit message: Pre-production check-in
Parts:
- J1, J2, J3, J4: footprint TerminalBlock_Phoenix:TerminalBlock_Phoenix_MPT-0,5-3-2.54_1x03_P2.54mm_Horizontal -> Connector_PinHeader_2.54mm:PinHeader_1x03_P2.54mm_Horizontal
- J5, J6, J7: footprint TerminalBlock_Phoenix:TerminalBlock_Phoenix_MPT-0,5-4-2.54_1x04_P2.54mm_Horizontal -> Connector_PinHeader_2.54mm:PinHeader_1x04_P2.54mm_Horizontal
- J8: footprint TerminalBlock_Phoenix:TerminalBlock_Phoenix_MPT-0,5-2-2.54_1x02_P2.54mm_Horizontal -> Connector_PinHeader_2.54mm:PinHeader_1x02_P2.54mm_Horizontal
Connections:
- net RXDI_NFC_5: now also J6.2 (Pin_2); no longer J6.3 (Pin_3)
- net SCL_DISP_5: now also J7.2 (Pin_2); no longer J7.3 (Pin_3)
- net SDA_DISP_5: now also J7.3 (Pin_3); no longer J7.2 (Pin_2)
- net TXDO_NFC_5: now also J6.3 (Pin_3); no longer J6.2 (Pin_2)
- net WG_D0_5: now also J5.3 (Pin_3); no longer J5.2 (Pin_2)
- net WG_D1_5: now also J5.2 (Pin_2); no longer J5.3 (Pin_3)
- net +BATT renamed +12V
